Commit message: Update rrbot.urdf
Updated.

File: rrbot.urdf (robot description, URDF)
Before this commit: robot RRbot, 6 links, 5 joints
Links:
- link RRbot_hokuyo_link: geometry collision box size=0.1 0.1 0.1; visual box size=0.1 0.1 0.1

Commit message: Update rrbot.urdf

File: rrbot.urdf (robot description, URDF)
Before this commit: robot RRbot, 6 links, 5 joints
Links:
- removed link RRbot_camera_link
- removed link RRbot_hokuyo_link
- removed link RRbot_link1
- removed link RRbot_link2
- removed link RRbot_link3
- added link rr_bot_camera_link, mass 1e-5; collision box size=0.05 0.05 0.05; visual box size=0.05 0.05 0.05
- added link rr_bot_hokuyo_link, mass 1e-5; collision box size=0.1 0.1 0.1; visual box size=0.1 0.1 0.1
- added link rr_bot_link1, mass 1; collision box size=0.1 0.1 2; visual box size=0.1 0.1 2
- added link rr_bot_link2, mass 1; collision box size=0.1 0.1 1; visual box size=0.1 0.1 1
- added link rr_bot_link3, mass 1; collision box size=0.1 0.1 1; visual box size=0.1 0.1 1
Joints:
- removed joint RRbot_camera_joint
- removed joint RRbot_fixed
- removed joint RRbot_hokuyo_joint
- removed joint RRbot_joint1
- removed joint RRbot_joint2
- added joint rr_bot_camera_joint: type fixed, parent rr_bot_link3, child rr_bot_camera_link, origin xyz=0.05 0 0.9 rpy=0 0 0, axis 0 1 0
- added joint rr_bot_fixed: type fixed, parent world, child rr_bot_link1, origin xyz=0 0 0 rpy=0 0 0
- added joint rr_bot_hokuyo_joint: type fixed, parent rr_bot_link3, child rr_bot_hokuyo_link, origin xyz=0 0 0.975 rpy=0 0 0, axis 0 1 0
- added joint rr_bot_joint1: type revolute, parent rr_bot_link1, child rr_bot_link2, origin xyz=0 0.1 1.95 rpy=0 0 0, axis 0 1 0
- added joint rr_bot_joint2: type revolute, parent rr_bot_link2, child rr_bot_link3, origin xyz=0 0.1 0.9 rpy=0 0 0, axis 0 1 0
